Commit message: Modify the height of camera and lidar to match the actual robot in real-life specs

File: urdf/turtlebot3_burger.urdf (robot description, URDF)
Before this commit: robot turtlebot3_burger, 12 links, 11 joints
Joints:
- joint scan_joint: origin xyz=-0.033 0 0.122 rpy=0 0 0 -> xyz=-0.033 0 0.715 rpy=0 0 0
